Commit message: Added basic Gazebo sim

File: description/mobile_robot.xacro (robot description, xacro)
@@ -56,4 +56,7 @@
        </xacro:inertial_box>
    </link>
+   <gazebo reference="chassis">
+    <material>Gazebo/White</material>
+   </gazebo>
    <!-- LEFT WHEEL LINK -->
    <joint name="left_wheel_joint" type="continuous">
@@ -80,4 +83,7 @@
         </xacro:inertial_cylinder>
   </link>
+  <gazebo reference="left_wheel">
+    <material>Gazebo/Blue</material>
+  </gazebo>
 <!-- RIGHT WHEEL LINK -->
 <joint name="right_wheel_joint" type="continuous">
@@ -104,4 +110,7 @@
         </xacro:inertial_cylinder>
   </link>
+  <gazebo reference="right_wheel">
+    <material>Gazebo/Blue</material>
+  </gazebo>
   <!-- CASTER WHEEL LINK -->
   <joint name="caster_wheel_joint" type="fixed">
@@ -127,3 +136,8 @@
     </xacro:inertial_sphere>
   </link>
+  <gazebo reference="caster_wheel">
+    <material>Gazebo/Black</material>
+    <mu1 value="0.001"/>
+    <mu2 value="0.001"/>
+  </gazebo>
 </robot>

File: description/robot.urdf.xacro (robot description, xacro)
@@ -2,3 +2,4 @@
 <robot xmlns:xacro="http://www.ros.org/wiki/xacro"  name="robot">
     <xacro:include filename="mobile_robot.xacro" />
+    <xacro:include filename="gazebo_control.xacro" />
 </robot>
